File: FormulaMixer_PCB/FormulaMixer_PCB-rounded.kicad_pcb (KiCad board)
At the start: 4 copper layers, 74.5 x 76.8 mm, 45 parts, among them J1 Conn_01x04, J2 Conn_01x04, J3 Conn_01x04, J4 Conn_01x04, J5 Conn_01x02, Q1 BC847, Q2 BC847, SW1 RotaryEncoder_Switch, SW2 SW_Push, SW3 SW_Push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

Commit message: Annotate PCB some, add mounting holes
Parts:
- added G***: LOGO, Connector_JST_Downloaded:earth_small, B.Cu at (89.8, 77.2)
- added REF**: MountingHole_3.2mm_M3, MountingHole:MountingHole_3.2mm_M3, F.Cu at (121.5, 115.0)
- added REF**: MountingHole_3.2mm_M3, MountingHole:MountingHole_3.2mm_M3, F.Cu at (58.5, 115.0)
- added REF**: MountingHole_3.2mm_M3, MountingHole:MountingHole_3.2mm_M3, F.Cu at (58.8, 46.0)
- added REF**: MountingHole_3.2mm_M3, MountingHole:MountingHole_3.2mm_M3, F.Cu at (121.5, 46.0)
- J1: value Conn_01x04 -> Pump1
- J2: value Conn_01x04 -> Pump2
- J3: value Conn_01x04 -> Pump3
- J4: value Conn_01x04 -> Pump4
- J5: value Conn_01x02 -> +12V GND
Other:
- board text added: "Formula Mixer Main Board Designed on Earth"
